File: circuit/KiCad/agccs-ctrl22.kicad_pcb (KiCad board)
At the start: 2 copper layers, 86.5 x 103 mm, 103 parts, among them J1 Screw_Terminal_01x05, J2 Screw_Terminal_01x05, J3 Conn_01x04, J4 Conn_01x04, J5 Conn_02x04_Top_Bottom, J6 Screw_Terminal_01x09, J7 Screw_Terminal_01x09, Q1 BSS138, U1 AQH3223, U10 ATmega4808-X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

Commit message: qe
Other:
- board text added: "AGCCS-Ctrl22 Rev1.2 02/2021"
- board text removed: "FGCCS-Ctrl22 Rev1.1 08/2020"

Commit message: fx
Parts:
- D12: value B220 -> PMEG4010BEA; footprint Diode_SMD:D_SMB_Handsoldering -> Diode_SMD:D_SOD-323_HandSoldering
- moved D12 2.56 mm to (154.9, 85.1)
Routing:
- net GND: track 574.5 -> 679.3 mm, vias 51 -> 54
- net Net-(D12-Pad1): track 14.2 -> 13.1 mm
- net /ATmega4808 and Peripherals/IO0: track 51.5 -> 52.4 mm
- net (no net): track 0.85 -> 0.00 mm, vias 1 -> 0
- net +12V: track 197.2 -> 196.6 mm, vias 5 -> 4

Commit message: tm
Parts:
- moved D6 0.56 mm to (171.8, 88.4)
Routing:
- net GND: track 679.3 -> 677.6 mm
- net /ATmega4808 and Peripherals/Button: track 45.3 -> 46.4 mm
- net Net-(R23-Pad1): track 30.2 -> 31.3 mm
- net /ATmega4808 and Peripherals/Lock_State: track 34.1 -> 34.8 mm
- net +3V3: vias 20 -> 19

Commit message: qe
Parts:
- added C27: 2200u16V, Capacitor_THT:CP_Radial_D12.5mm_P7.50mm, B.Cu at (157.1, 77.9)
- added D13: 9.1, Diode_SMD:D_SOD-323_HandSoldering, F.Cu at (115.1, 141.8)
- added R40: 2k, Resistor_SMD:R_0603_1608Metric_Pad1.05x0.95mm_HandSolder, F.Cu at (110.0, 142.1)
- added R41: 1k, Resistor_SMD:R_0603_1608Metric_Pad1.05x0.95mm_HandSolder, F.Cu at (112.0, 142.1)
- added U14: LM321LV, Package_TO_SOT_SMD:SOT-23-5, F.Cu at (175.4, 59.6)
- R11: value 10k -> 2k
- R12: value 31.6k -> 5.6k
- moved R27 72.3 mm to (175.4, 54.6)
- moved R26 70.1 mm to (175.4, 56.6), turned to 180 degrees
- moved U7 10.5 mm to (176.0, 65.8)
- moved C14 10.2 mm to (179.6, 61.5), turned to 0 degrees
- moved J4 9.47 mm to (121.2, 142.5), turned to 270 degrees
- moved R37 7.02 mm to (129.0, 136.4), turned to 180 degrees
- moved R38 6.99 mm to (129.0, 138.9), turned to 180 degrees
- moved R34 6.98 mm to (129.1, 133.9), turned to 180 degrees
- moved R6 5.63 mm to (149.7, 90.9)
- moved F2 5.55 mm to (114.0, 48.0)
- moved R3 5.46 mm to (144.1, 90.9)
- moved C12 2.16 mm to (145.4, 96.4)
- moved R5 2.06 mm to (148.0, 90.9)
- moved R4 1.75 mm to (146.1, 90.9)
- moved C17 1.71 mm to (148.2, 101.5)
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Connections:
- net /ATmega4808 and Peripherals/12V_sep renamed +12P
- J3 pad 1: +12V -> GND
- J3 pad 2: /ATmega4808 and Peripherals/ATmega_RX2 -> /ATmega4808 and Peripherals/ATmega_TX2
- J3 pad 3: /ATmega4808 and Peripherals/ATmega_TX2 -> /ATmega4808 and Peripherals/ATmega_RX2
- J3 pad 4: GND -> +12V
- R26 pad 2: /Analog Section and Low Voltage Outputs/BIAS -> Net-(R26-Pad2)
- R27 pad 1: /Analog Section and Low Voltage Outputs/BIAS -> Net-(R26-Pad2)
Routing:
- net /Analog Section and Low Voltage Outputs/BIAS: track 54.3 -> 107.5 mm, vias 0 -> 2
- net Net-(F2-Pad1): track 52.1 -> 78.4 mm, vias 0 -> 2
- net GND: track 677.6 -> 694.3 mm, vias 54 -> 46
- net /ATmega4808 and Peripherals/RS485_A: track 11.1 -> 26.1 mm, vias 2 -> 0
- net /ATmega4808 and Peripherals/RS485_B: track 8.13 -> 20.0 mm
- net +12V: track 196.6 -> 206.9 mm
- net /ATmega4808 and Peripherals/ESP_IO12: track 49.0 -> 41.6 mm
- net /ATmega4808 and Peripherals/RS485_RX: track 59.0 -> 51.9 mm
- net /ATmega4808 and Peripherals/ATmega_TX0: track 57.1 -> 63.3 mm, vias 1 -> 2
- net /ATmega4808 and Peripherals/BOT: track 0.00 -> 5.08 mm
- net /ATmega4808 and Peripherals/RS485_TX: track 53.5 -> 48.7 mm
- net +12P: track 62.5 -> 58.2 mm
- net +3V3: track 302.6 -> 298.4 mm
- net /ATmega4808 and Peripherals/RS485_XDIR: track 62.0 -> 66.2 mm
- net Net-(R26-Pad2): track 0.00 -> 4.13 mm
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
Commit message: qe
Parts:
- removed D11: BAT54S, Package_TO_SOT_SMD:SOT-23_Handsoldering
- C12: value 10000u16V -> 15000u16V
- R13: value 40.2k -> 62k
- R24: value 5.6K -> 5.6k
- moved R40 0.64 mm to (109.3, 142.1)
- moved R39 0.38 mm to (179.4, 74.5)
- moved R34 0.13 mm to (129.0, 133.9)
Routing:
- net +3V3: track 298.4 -> 288.8 mm
- net GND: track 694.3 -> 686.7 mm
- net /ATmega4808 and Peripherals/CP: track 51.0 -> 47.5 mm

Commit message: qe
Parts:
- added C28: 100n, Capacitor_SMD:C_0805_2012Metric_Pad1.18x1.45mm_HandSolder, F.Cu at (175.5, 51.6)
- J5: value Conn_02x04_Top_Bottom -> Conn_02x04
- R39: footprint Resistor_SMD:R_0603_1608Metric_Pad0.98x0.95mm_HandSolder -> Resistor_SMD:R_0603_1608Metric_Pad1.05x0.95mm_HandSolder
- moved R33 14.3 mm to (184.0, 137.3), turned to 270 degrees
- moved R32 7.46 mm to (183.9, 127.0), turned to 270 degrees
- moved R31 4.46 mm to (183.9, 117.0), turned to 270 degrees
- moved R30 3.53 mm to (179.2, 122.9)
- moved R29 3.51 mm to (179.1, 119.8)
- moved R28 3.48 mm to (179.1, 117.0)
- moved C25 2.61 mm to (174.1, 122.9)
- moved C24 2.56 mm to (174.1, 119.8)
- moved C23 2.42 mm to (174.1, 117.1)
Connections:
- J5 pad 2: /ATmega4808 and Peripherals/ESP_TX0 -> GND
- J5 pad 3: /ATmega4808 and Peripherals/ESP_RX0 -> /ATmega4808 and Peripherals/ESP_TX0
- J5 pad 4: /ATmega4808 and Peripherals/IO0 -> +3V3
- J5 pad 5: GND -> /ATmega4808 and Peripherals/ESP_RX0
- J5 pad 6: +3V3 -> /ATmega4808 and Peripherals/ESP_IO15
- J5 pad 7: /ATmega4808 and Peripherals/ESP_IO15 -> /ATmega4808 and Peripherals/IO0
Routing:
- net +12V: track 206.9 -> 197.1 mm, vias 4 -> 5
- net /Analog Section and Low Voltage Outputs/CT0_L: track 12.4 -> 7.89 mm
- net /ATmega4808 and Peripherals/CT0: track 63.9 -> 67.7 mm, vias 4 -> 3
- net Net-(C28-Pad1): track 4.13 -> 7.42 mm
- net GND: track 686.7 -> 690.0 mm
- net /ATmega4808 and Peripherals/CT2: track 50.5 -> 53.4 mm, vias 4 -> 3
- net /ATmega4808 and Peripherals/CT1: track 58.2 -> 60.6 mm, vias 4 -> 3
- net /Analog Section and Low Voltage Outputs/BIAS: track 107.5 -> 108.8 mm
- net /Analog Section and Low Voltage Outputs/CT1_L: track 12.0 -> 11.1 mm, vias 2 -> 0
- net /Analog Section and Low Voltage Outputs/CT2_L: track 17.8 -> 18.5 mm, vias 2 -> 0
- net /ATmega4808 and Peripherals/BOT: track 5.08 -> 5.72 mm
Other:
- board text added: "12V"
- board text added: "GND"

Commit message: qe
Parts:
- C16: value 100u / 6.3V -> 100u6.3V
- C21: value 1n / 50V -> 1n50V
- C22: value 1u / 10V -> 1u10V
- moved D7 1.95 mm to (173.3, 78.1)
- moved R39 0.27 mm to (179.5, 74.8)
- moved F1 0.18 mm to (177.2, 47.1)
- moved R24 0.14 mm to (179.5, 77.3)
- renumbered RV3 to RV1, RV1 to RV3
Connections:
- net +12P renamed 12V_buffered
- net /ATmega4808 and Peripherals/ATmega_RESET renamed /ATmega4808 and Peripherals/AVR_RST
- net /ATmega4808 and Peripherals/ATmega_RX0 renamed /ATmega4808 and Peripherals/AVR_RX0
- net /ATmega4808 and Peripherals/ATmega_RX2 renamed /ATmega4808 and Peripherals/AVR_RX2
- net /ATmega4808 and Peripherals/ATmega_TX0 renamed /ATmega4808 and Peripherals/AVR_TX0
- net /ATmega4808 and Peripherals/ATmega_TX2 renamed /ATmega4808 and Peripherals/AVR_TX2
- net /ATmega4808 and Peripherals/EN renamed /ATmega4808 and Peripherals/ESP_EN
- net /ATmega4808 and Peripherals/IO0 renamed /ATmega4808 and Peripherals/ESP_IO0
- net /ATmega4808 and Peripherals/RS485_RX renamed /ATmega4808 and Peripherals/AVR_RX1
- net /ATmega4808 and Peripherals/RS485_TX renamed /ATmega4808 and Peripherals/AVR_TX1
- net /Analog Section and Low Voltage Outputs/12V_Fused renamed 12V_fused
- net Net-(F2-Pad1) renamed /Mains and Power Circuitry/L_fused
- net Net-(J5-Pad1) renamed /ATmega4808 and Peripherals/AVR_UDPI
- D7 pad 3: /ATmega4808 and Peripherals/Button -> Net-(D7-Pad3)
- J6 pad 5: /Analog Section and Low Voltage Outputs/Button_J6_5 -> /ATmega4808 and Peripherals/Button
- R24 pad 1: /Analog Section and Low Voltage Outputs/Button_J6_5 -> /ATmega4808 and Peripherals/Button
- R24 pad 2: /ATmega4808 and Peripherals/Button -> Net-(D7-Pad3)
- R39 pad 2: /ATmega4808 and Peripherals/Button -> Net-(D7-Pad3)
- U10 pad 10: /ATmega4808 and Peripherals/Button -> Net-(D7-Pad3)
Routing:
- net Net-(D7-Pad3): track 0.00 -> 45.1 mm, vias 0 -> 2
- net /ATmega4808 and Peripherals/Button: track 46.4 -> 11.6 mm, vias 2 -> 0
- net /Analog Section and Low Voltage Outputs/Button_J6_5: track 11.6 -> 0.00 mm
- net +3V3: track 288.8 -> 290.5 mm
- net GND: track 690.0 -> 691.5 mm

Commit message: qe
Parts:
- C1, C10, C11, C13, C14, C15, C17, C18, C2, C20, C23, C24, C25, C3, C4, C5, C6, C7, C8, C9: footprint Capacitor_SMD:C_0805_2012Metric_Pad1.15x1.40mm_HandSolder -> Capacitor_SMD:C_0805_2012Metric_Pad1.18x1.45mm_HandSolder
- moved R25 1.05 mm to (168.8, 127.4)
- moved C21 0.97 mm to (171.8, 127.5)
- moved R16 0.79 mm to (166.6, 104.8)
- moved R21 0.78 mm to (166.6, 102.1)
- moved R13 0.65 mm to (165.2, 79.2)
- moved C20 0.61 mm to (165.2, 77.2)
- moved R20 0.50 mm to (165.1, 82.0)
- moved R15 0.29 mm to (165.1, 84.8)
- moved C15 0.12 mm to (154.7, 109.9)
- moved C8 0.11 mm to (164.6, 66.4)
- moved U9 0.06 mm to (157.4, 125.6)
Connections:
- C23 pad 1: /ATmega4808 and Peripherals/CT0 -> /ATmega4808 and Peripherals/CT1
- C24 pad 1: /ATmega4808 and Peripherals/CT1 -> /ATmega4808 and Peripherals/CT2
- C25 pad 1: /ATmega4808 and Peripherals/CT2 -> /ATmega4808 and Peripherals/CT3
- D10 pad 3: /ATmega4808 and Peripherals/CT2 -> /ATmega4808 and Peripherals/CT3
- D8 pad 3: /ATmega4808 and Peripherals/CT0 -> /ATmega4808 and Peripherals/CT1
- D9 pad 3: /ATmega4808 and Peripherals/CT1 -> /ATmega4808 and Peripherals/CT2
- J4 pad 2: /ATmega4808 and Peripherals/AVR_TX0 -> /ATmega4808 and Peripherals/ESP_RX2
- J7 pad 4: /Analog Section and Low Voltage Outputs/CT0_L -> /Analog Section and Low Voltage Outputs/CT1_L
- J7 pad 6: /Analog Section and Low Voltage Outputs/CT1_L -> /Analog Section and Low Voltage Outputs/CT2_L
- J7 pad 8: /Analog Section and Low Voltage Outputs/CT2_L -> /Analog Section and Low Voltage Outputs/CT3_L
- R28 pad 1: /ATmega4808 and Peripherals/CT0 -> /ATmega4808 and Peripherals/CT1
- R28 pad 2: /Analog Section and Low Voltage Outputs/CT0_L -> /Analog Section and Low Voltage Outputs/CT1_L
- R29 pad 1: /ATmega4808 and Peripherals/CT1 -> /ATmega4808 and Peripherals/CT2
- R29 pad 2: /Analog Section and Low Voltage Outputs/CT1_L -> /Analog Section and Low Voltage Outputs/CT2_L
- R30 pad 1: /ATmega4808 and Peripherals/CT2 -> /ATmega4808 and Peripherals/CT3
- R30 pad 2: /Analog Section and Low Voltage Outputs/CT2_L -> /Analog Section and Low Voltage Outputs/CT3_L
- R31 pad 1: /Analog Section and Low Voltage Outputs/CT0_L -> /Analog Section and Low Voltage Outputs/CT1_L
- R32 pad 1: /Analog Section and Low Voltage Outputs/CT1_L -> /Analog Section and Low Voltage Outputs/CT2_L
- R33 pad 1: /Analog Section and Low Voltage Outputs/CT2_L -> /Analog Section and Low Voltage Outputs/CT3_L
- U10 pad 11: /ATmega4808 and Peripherals/CT0 -> /ATmega4808 and Peripherals/CT1
- U10 pad 12: /ATmega4808 and Peripherals/CT1 -> /ATmega4808 and Peripherals/CT2
- U10 pad 13: /ATmega4808 and Peripherals/CT2 -> /ATmega4808 and Peripherals/CT3
Routing:
- net /ATmega4808 and Peripherals/CT0: track 67.7 -> 0.00 mm, vias 3 -> 0
- net /ATmega4808 and Peripherals/CT3: track 0.00 -> 53.4 mm, vias 0 -> 3
- net /Analog Section and Low Voltage Outputs/CT3_L: track 0.00 -> 18.5 mm
- net /ATmega4808 and Peripherals/ESP_RX2: track 55.3 -> 72.6 mm, vias 3 -> 4
- net /ATmega4808 and Peripherals/AVR_TX0: track 63.5 -> 50.7 mm
- net /Analog Section and Low Voltage Outputs/CT0_L: track 7.89 -> 0.00 mm
- net /Analog Section and Low Voltage Outputs/CT2_L: track 18.5 -> 11.1 mm
- net /ATmega4808 and Peripherals/CT2: track 53.4 -> 60.6 mm
- net /ATmega4808 and Peripherals/CT1: track 60.6 -> 67.7 mm
- net /Analog Section and Low Voltage Outputs/CT1_L: track 11.1 -> 7.89 mm
- net /ATmega4808 and Peripherals/ESP_EN: track 41.7 -> 43.4 mm
- net Net-(C28-Pad1): track 7.42 -> 8.54 mm
- net /Analog Section and Low Voltage Outputs/PP_to_relay: track 22.4 -> 23.2 mm
- net +12V: track 197.1 -> 197.7 mm
- net Net-(R23-Pad1): track 31.3 -> 30.7 mm
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