File: circuit/KiCad/agccs-ctrl22.kicad_pcb (KiCad board)
At the start: 2 copper layers, 86.5 x 103 mm, 108 parts, among them J1 Screw_Terminal_01x05, J2 Screw_Terminal_01x05, J3 Conn_01x04, J4 Conn_01x04, J5 Conn_02x04, J6 Screw_Terminal_01x09, J7 Screw_Terminal_01x09, Q1 BSS138, U1 AQH3223, U10 ATmega4808-X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

Commit message: qe
Routing:
- net /Mains and Power Circuitry/N: track 155.6 -> 137.0 mm, vias 2 -> 0
- net +12V: track 197.7 -> 206.0 mm, vias 5 -> 10
- net GND: track 691.8 -> 683.8 mm
- net Net-(Q1-Pad1): track 50.1 -> 56.6 mm
- net /Mains and Power Circuitry/L_fused: track 78.4 -> 81.0 mm, vias 2 -> 4
- net /Mains and Power Circuitry/C_L2: track 40.7 -> 42.6 mm, vias 1 -> 2
- net /ATmega4808 and Peripherals/AVR_TX0: track 50.7 -> 48.9 mm
- net +3V3: track 290.5 -> 289.8 mm
Other:
- board text added: "AGCCS-Ctrl22 Rev1.3 03/2021"
- board text removed: "AGCCS-Ctrl22 Rev1.2 02/2021"
