File: circuit/KiCad/analog_section_low_voltage.sch (KiCad schematic (older format))
At the start: 40 parts, among them J6 Screw_Terminal_01x09, J7 Screw_Terminal_01x09, U11 LM7332, U12 CPC1114N, U13 CPC1114N

Commit message: qe
Parts:
- added U14: LM321LV, Package_TO_SOT_SMD:SOT-23-5, symbol Amplifier_Operational:LM321
- R39: footprint Resistor_SMD:R_0603_1608Metric_Pad0.98x0.95mm_HandSolder -> Resistor_SMD:R_0603_1608Metric_Pad1.05x0.95mm_HandSolder
Connections:
- net +3V3: now also U14.5 (V+)
- net BIAS: now also U14.3 (-), U14.4; no longer R26.2, R27.1
- net GND: now also U14.2 (V-)
- new net: R26.2, R27.1, U14.1 (+)
Other:
- moved on the sheet: C23, C24, C25, D10, D8, D9, R26, R27, R28, R29, R30, R31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

Commit message: qe
Parts:
- removed D11: BAT54S, Package_TO_SOT_SMD:SOT-23_Handsoldering, symbol Diode:BAT54S
- D10, D8, D9: PartNo (none) -> 757-TBAT54SLM; Supplier (none) -> Mouser
- D5, D7: PartNo 583-BAT54S -> 757-TBAT54SLM
- R13: value 40.2k -> 62k; PartNo 594-MCT06030C4022FP5 -> 594-MCT06030C6202FP5
- R24: value 5.6K -> 5.6k; PartNo 594-MCT06030C1000FP5 -> 594-MCT06030C5601FP5
Changed lines of the file:
@@
 Wire Wire Line
 	6050 3000 6150 3000
-Text HLabel 3050 2900 0    50   Input ~ 0
+Text HLabel 3650 2900 0    50   Input ~ 0
 PWM_Out
 $Comp
@@
 L power:GND #PWR0106
 U 1 1 5E91FFF3
-P 3600 3750
-F 0 "#PWR0106" H 3600 3500 50  0001 C CNN
-F 1 "GND" H 3605 3577 50  0000 C CNN
-F 2 "" H 3600 3750 50  0001 C CNN
-F 3 "" H 3600 3750 50  0001 C CNN
-	1    3600 3750
-	1    0    0    -1
-$EndComp
-Text HLabel 3050 1800 0    50   Output ~ 0
+P 4050 3750
+F 0 "#PWR0106" H 4050 3500 50  0001 C CNN
+F 1 "GND" H 4055 3577 50  0000 C CNN
+F 2 "" H 4050 3750 50  0001 C CNN
+F 3 "" H 4050 3750 50  0001 C CNN
+	1    4050 3750
+	1    0    0    -1
+$EndComp
+Text HLabel 3600 1800 0    50   Output ~ 0
 CP
 Wire Wire Line
@@
 P 4300 1800
 F 0 "R13" V 4400 1750 50  0000 L CNN
-F 1 "40.2k" V 4500 1750 50  0000 L CNN
+F 1 "62k" V 4500 1750 50  0000 L CNN
 F 2 "Resistor_SMD:R_0603_1608Metric_Pad1.05x0.95mm_HandSolder" H 4300 1800 50  0001 C CNN
 F 3 "~" H 4300 1800 50  0001 C CNN
 F 4 "" H 4300 1800 50  0001 C CNN "Part"
-F 5 "594-MCT06030C4022FP5 " H 4300 1800 50  0001 C CNN "PartNo"
+F 5 " 594-MCT06030C6202FP5 " H 4300 1800 50  0001 C CNN "PartNo"
 F 6 "Mouser" H 4300 1800 50  0001 C CNN "Supplier"
 	1    4300 1800
@@
 F 3 "https://www.diodes.com/assets/Datasheets/ds11005.pdf" H 4980 5200 50  0001 C CNN
 F 4 "" H 5100 5200 50  0001 C CNN "Part"
-F 5 "583-BAT54S " H 5100 5200 50  0001 C CNN "PartNo"
+F 5 " 757-TBAT54SLM " H 5100 5200 50  0001 C CNN "PartNo"
 F 6 "Mouser" H 5100 5200 50  0001 C CNN "Supplier"
 	1    5100 5200
@@
 F 3 "https://www.diodes.com/assets/Datasheets/ds11005.pdf" H 6180 5200 50  0001 C CNN
 F 4 "" H 6300 5200 50  0001 C CNN "Part"
-F 5 "583-BAT54S " H 6300 5200 50  0001 C CNN "PartNo"
+F 5 " 757-TBAT54SLM " H 6300 5200 50  0001 C CNN "PartNo"
 F 6 "Mouser" H 6300 5200 50  0001 C CNN "Supplier"
 	1    6300 5200
@@
 P 6950 4600
 F 0 "R24" V 7000 4750 50  0000 C CNN
-F 1 "5.6K" V 6845 4600 50  0000 C CNN
+F 1 "5.6k" V 6845 4600 50  0000 C CNN
 F 2 "Resistor_SMD:R_0603_1608Metric_Pad1.05x0.95mm_HandSolder" H 6950 4600 50  0001 C CNN
 F 3 "~" H 6950 4600 50  0001 C CNN
 F 4 "" H 6950 4600 50  0001 C CNN "Part"
-F 5 "594-MCT06030C1000FP5 " H 6950 4600 50  0001 C CNN "PartNo"
+F 5 "594-MCT06030C5601FP5 " H 6950 4600 50  0001 C CNN "PartNo"
 F 6 "Mouser" H 6950 4600 50  0001 C CNN "Supplier"
 	1    6950 4600
@@
 F 2 "Package_TO_SOT_SMD:SOT-23_Handsoldering" H 3275 5625 50  0001 L CNN
 F 3 "https://www.diodes.com/assets/Datasheets/ds11005.pdf" H 3080 5500 50  0001 C CNN
+F 4 " 757-TBAT54SLM " H 3200 5500 50  0001 C CNN "PartNo"
+F 5 "Mouser" H 3200 5500 50  0001 C CNN "Supplier"
 	1    3200 5500
 	0    1    -1   0
@@
 F 2 "Package_TO_SOT_SMD:SOT-23_Handsoldering" H 3275 6525 50  0001 L CNN
 F 3 "https://www.diodes.com/assets/Datasheets/ds11005.pdf" H 3080 6400 50  0001 C CNN
+F 4 " 757-TBAT54SLM " H 3200 6400 50  0001 C CNN "PartNo"
+F 5 "Mouser" H 3200 6400 50  0001 C CNN "Supplier"
 	1    3200 6400
 	0    1    -1   0
@@
 F 2 "Package_TO_SOT_SMD:SOT-23_Handsoldering" H 3275 7425 50  0001 L CNN
 F 3 "https://www.diodes.com/assets/Datasheets/ds11005.pdf" H 3080 7300 50  0001 C CNN
+F 4 " 757-TBAT54SLM " H 3200 7300 50  0001 C CNN "PartNo"
+F 5 "Mouser" H 3200 7300 50  0001 C CNN "Supplier"
 	1    3200 7300
 	0    1    -1   0
@@
 	-1   0    0    -1
 $EndComp
-$Comp
-L Diode:BAT54S D11
-U 1 1 5F4367A4
-P 3600 2150
-F 0 "D11" V 3646 2238 50  0000 L CNN
-F 1 "BAT54S" V 3555 2238 50  0000 L CNN
-F 2 "Package_TO_SOT_SMD:SOT-23_Handsoldering" H 3675 2275 50  0001 L CNN
-F 3 "https://www.diodes.com/assets/Datasheets/ds11005.pdf" H 3480 2150 50  0001 C CNN
-	1    3600 2150
-	0    1    -1   0
-$EndComp
 Wire Wire Line
 	8500 2600 9250 2600
@@
 Wire Wire Line
 	4050 1800 4050 3400
-Wire Wire Line
-	3600 2450 3600 3750
-Wire Wire Line
-	3600 3750 4050 3750
-Wire Wire Line
-	3050 1800 3400 1800
-Wire Wire Line
-	3600 1850 3600 1150
-Wire Wire Line
-	3600 1150 4050 1150
-Connection ~ 4050 1150
-Wire Wire Line
-	3400 2150 3400 1800
-Connection ~ 3400 1800
-Wire Wire Line
-	3400 1800 4050 1800
 Wire Wire Line
 	4650 3600 4650 3750
@@
 $EndComp
 Wire Wire Line
-	3050 2900 4800 2900
+	3650 2900 4800 2900
 Wire Wire Line
 	4650 2650 4650 3100
 Connection ~ 4650 3100
-Connection ~ 3600 3750
 $Comp
 L Device:R_Small R39
@@
 Wire Wire Line
 	1550 4150 2300 4150
+Wire Wire Line
+	3600 1800 4050 1800
 $EndSCHEMATC

Commit message: qe
Parts:
- added C28: 100n, Capacitor_SMD:C_0805_2012Metric_Pad1.18x1.45mm_HandSolder, symbol Device:C_Small
Connections:
- net GND: now also C28.2
- net at R26.2, R27.1, U14.1 (+): now also C28.1
Other:
- moved on the sheet: R26, R27
Changed lines of the file:
@@
 L Device:R_Small R27
 U 1 1 5EC624D0
-P 1250 3950
-F 0 "R27" H 1309 3996 50  0000 L CNN
-F 1 "10k" H 1309 3905 50  0000 L CNN
-F 2 "Resistor_SMD:R_0603_1608Metric_Pad1.05x0.95mm_HandSolder" H 1250 3950 50  0001 C CNN
-F 3 "~" H 1250 3950 50  0001 C CNN
-F 4 "" H 1250 3950 50  0001 C CNN "Part"
-F 5 "594-MCT06030C1002FP5 " H 1250 3950 50  0001 C CNN "PartNo"
-F 6 "Mouser" H 1250 3950 50  0001 C CNN "Supplier"
-	1    1250 3950
+P 850 3950
+F 0 "R27" H 909 3996 50  0000 L CNN
+F 1 "10k" H 909 3905 50  0000 L CNN
+F 2 "Resistor_SMD:R_0603_1608Metric_Pad1.05x0.95mm_HandSolder" H 850 3950 50  0001 C CNN
+F 3 "~" H 850 3950 50  0001 C CNN
+F 4 "" H 850 3950 50  0001 C CNN "Part"
+F 5 "594-MCT06030C1002FP5 " H 850 3950 50  0001 C CNN "PartNo"
+F 6 "Mouser" H 850 3950 50  0001 C CNN "Supplier"
+	1    850  3950
 	1    0    0    -1
 $EndComp
@@
 L Device:R_Small R26
 U 1 1 5EC624D6
-P 1250 3600
-F 0 "R26" H 1309 3646 50  0000 L CNN
-F 1 "10k" H 1309 3555 50  0000 L CNN
-F 2 "Resistor_SMD:R_0603_1608Metric_Pad1.05x0.95mm_HandSolder" H 1250 3600 50  0001 C CNN
-F 3 "~" H 1250 3600 50  0001 C CNN
-F 4 "" H 1250 3600 50  0001 C CNN "Part"
-F 5 "594-MCT06030C1002FP5 " H 1250 3600 50  0001 C CNN "PartNo"
-F 6 "Mouser" H 1250 3600 50  0001 C CNN "Supplier"
-	1    1250 3600
+P 850 3600
+F 0 "R26" H 909 3646 50  0000 L CNN
+F 1 "10k" H 909 3555 50  0000 L CNN
+F 2 "Resistor_SMD:R_0603_1608Metric_Pad1.05x0.95mm_HandSolder" H 850 3600 50  0001 C CNN
+F 3 "~" H 850 3600 50  0001 C CNN
+F 4 "" H 850 3600 50  0001 C CNN "Part"
+F 5 "594-MCT06030C1002FP5 " H 850 3600 50  0001 C CNN "PartNo"
+F 6 "Mouser" H 850 3600 50  0001 C CNN "Supplier"
+	1    850  3600
 	1    0    0    -1
 $EndComp
@@
 $EndComp
 Wire Wire Line
-	1250 3700 1250 3750
-Wire Wire Line
-	1250 3750 1550 3750
-Connection ~ 1250 3750
-Wire Wire Line
-	1250 3750 1250 3850
-Wire Wire Line
-	1250 4050 1250 4250
+	850  3700 850  3750
+Connection ~ 850  3750
+Wire Wire Line
+	850  3750 850  3850
+Wire Wire Line
+	850  4050 850  4250
 Wire Wire Line
 	1750 4150 1750 4250
 Wire Wire Line
 	1750 4250 1250 4250
-Connection ~ 1250 4250
 Wire Wire Line
 	1750 3550 1750 3400
 Wire Wire Line
 	1750 3400 1250 3400
-Connection ~ 1250 3400
-Wire Wire Line
-	1250 3400 1250 3500
+Wire Wire Line
+	850  3400 850  3500
 Wire Wire Line
 	1550 4150 1550 3950
 Wire Wire Line
-	2150 3850 2300 3850
-Wire Wire Line
-	2300 4150 2300 3850
-Connection ~ 2300 3850
-Wire Wire Line
-	2300 3850 2450 3850
+	2150 3850 2200 3850
+Wire Wire Line
+	2200 4150 2200 3850
+Connection ~ 2200 3850
+Wire Wire Line
+	2200 3850 2450 3850
 Wire Notes Line
 	2950 4550 2950 3150
@@
 Button
 Wire Wire Line
-	1550 4150 2300 4150
-Wire Wire Line
 	3600 1800 4050 1800
+Connection ~ 1250 3400
+Connection ~ 1250 4250
+Wire Wire Line
+	2550 5250 2550 5350
+$Comp
+L Device:C_Small C?
+U 1 1 604D0F1E
+P 1250 3950
+AR Path="/5E98FA8A/604D0F1E" Ref="C?"  Part="1"
+AR Path="/5E903BF9/604D0F1E" Ref="C28"  Part="1"
+F 0 "C28" H 1342 3996 50  0000 L CNN
+F 1 "100n" H 1342 3905 50  0000 L CNN
+F 2 "Capacitor_SMD:C_0805_2012Metric_Pad1.18x1.45mm_HandSolder" H 1250 3950 50  0001 C CNN
+F 3 "~" H 1250 3950 50  0001 C CNN
+F 4 "" H 1250 3950 50  0001 C CNN "Part"
+F 5 "963-EMF212B7104KGHT " H 1250 3950 50  0001 C CNN "PartNo"
+F 6 "Mouser" H 1250 3950 50  0001 C CNN "Supplier"
+	1    1250 3950
+	1    0    0    -1
+$EndComp
+Wire Wire Line
+	850  3750 1250 3750
+Wire Wire Line
+	850  3400 1250 3400
+Wire Wire Line
+	850  4250 1250 4250
+Wire Wire Line
+	1250 3850 1250 3750
+Connection ~ 1250 3750
+Wire Wire Line
+	1250 3750 1550 3750
+Wire Wire Line
+	1250 4050 1250 4250
+Wire Wire Line
+	1550 4150 2200 4150
 $EndSCHEMATC

Commit message: qe
Parts:
- U14: PartNo (none) -> 595-LM321LVIDBVR; Supplier (none) -> Mouser
Changed lines of the file:
@@
 F 2 "Package_TO_SOT_SMD:SOT-23-5" H 1850 3850 50  0001 C CNN
 F 3 "http://www.ti.com/lit/ds/symlink/lm321.pdf" H 1850 3850 50  0001 C CNN
+F 4 "595-LM321LVIDBVR" H 1850 3850 50  0001 C CNN "PartNo"
+F 5 "Mouser" H 1850 3850 50  0001 C CNN "Supplier"
 	1    1850 3850
 	1    0    0    -1

Commit message: qe
Parts:
- removed D7: BAT54S, Package_TO_SOT_SMD:SOT-23_Handsoldering, symbol Diode:BAT54S
- removed F1: FSMD020, Fuse:Fuse_1812_4532Metric_Pad1.30x3.40mm_HandSolder, symbol Device:Polyfuse_Small
- removed R24: 5.6k, Resistor_SMD:R_0603_1608Metric_Pad1.05x0.95mm_HandSolder, symbol Device:R_Small
- removed R39: 2k, Resistor_SMD:R_0603_1608Metric_Pad1.05x0.95mm_HandSolder, symbol Device:R_Small
Connections:
- net Button_J6_5 is gone; now on net Button: J6.5 (Pin_5)
- net 12V_Fused renamed 12V_fused
Other:
- moved on the sheet: C18, C19, C20, C23, C24, C25, C28, D10, D5, D6, D8, D9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

Commit message: qe
Parts:
- C18, C20, C23, C24, C25: footprint Capacitor_SMD:C_0805_2012Metric_Pad1.15x1.40mm_HandSolder -> Capacitor_SMD:C_0805_2012Metric_Pad1.18x1.45mm_HandSolder
- J7: PartNo (none) -> 490-TB004-508-18BE
- U11: symbol Device:Opamp_Dual_Generic -> agccs-ctrl22:Opamp_Dual_Generic_SmallVcc
Connections:
- net CT0 is gone; now on net CT1: C23.1, D8.3, R28.1
- net CT0_L is gone; now on net CT1_L: J7.4 (Pin_4), R28.2, R31.1
- net CT1: no longer C24.1, D9.3, R29.1
- net CT1_L: no longer J7.6 (Pin_6), R29.2, R32.1
- net CT2: now also C24.1, D9.3, R29.1; no longer C25.1, D10.3, R30.1
- net CT2_L: now also J7.6 (Pin_6), R29.2, R32.1; no longer J7.8 (Pin_8), R30.2, R33.1
- new net CT3: C25.1, D10.3, R30.1
- new net CT3_L: J7.8 (Pin_8), R30.2, R33.1
Changed lines of the file:
@@
 F 0 "C20" H 8592 1346 50  0000 L CNN
 F 1 "100n" H 8592 1255 50  0000 L CNN
-F 2 "Capacitor_SMD:C_0805_2012Metric_Pad1.15x1.40mm_HandSolder" H 8500 1300 50  0001 C CNN
+F 2 "Capacitor_SMD:C_0805_2012Metric_Pad1.18x1.45mm_HandSolder" H 8500 1300 50  0001 C CNN
 F 3 "~" H 8500 1300 50  0001 C CNN
 F 4 "" H 8500 1300 50  0001 C CNN "Part"
@@
 $EndComp
 $Comp
-L Device:Opamp_Dual_Generic U11
+L agccs-ctrl22:Opamp_Dual_Generic_SmallVcc U11
 U 3 1 5E913947
 P 8100 1800
@@
 F 0 "C18" H 8392 2296 50  0000 L CNN
 F 1 "100n" H 8392 2205 50  0000 L CNN
-F 2 "Capacitor_SMD:C_0805_2012Metric_Pad1.15x1.40mm_HandSolder" H 8300 2250 50  0001 C CNN
+F 2 "Capacitor_SMD:C_0805_2012Metric_Pad1.18x1.45mm_HandSolder" H 8300 2250 50  0001 C CNN
 F 3 "~" H 8300 2250 50  0001 C CNN
 F 4 "" H 8300 2250 50  0001 C CNN "Part"
@@
 Text HLabel 7450 4400 0    50   Output ~ 0
 PP
-Text HLabel 1475 6400 0    50   Input ~ 0
-Signal_Relay
 Wire Notes Line
 	7350 800  7350 2450
@@
 PP_to_relay
 Text HLabel 4525 1625 2    50   Output ~ 0
-CT0
+CT1
 $Comp
 L power:GND #PWR?
@@
 F 0 "C23" H 3717 2021 50  0000 L CNN
 F 1 "100n" H 3717 1930 50  0000 L CNN
-F 2 "Capacitor_SMD:C_0805_2012Metric_Pad1.15x1.40mm_HandSolder" H 3625 1975 50  0001 C CNN
+F 2 "Capacitor_SMD:C_0805_2012Metric_Pad1.18x1.45mm_HandSolder" H 3625 1975 50  0001 C CNN
 F 3 "~" H 3625 1975 50  0001 C CNN
 F 4 "" H 3625 1975 50  0001 C CNN "Part"
@@
 $EndComp
 Text HLabel 4525 2875 2    50   Output ~ 0
-CT1
+CT2
 $Comp
 L Device:C_Small C?
@@
 F 0 "C24" H 3717 3271 50  0000 L CNN
 F 1 "100n" H 3717 3180 50  0000 L CNN
-F 2 "Capacitor_SMD:C_0805_2012Metric_Pad1.15x1.40mm_HandSolder" H 3625 3225 50  0001 C CNN
+F 2 "Capacitor_SMD:C_0805_2012Metric_Pad1.18x1.45mm_HandSolder" H 3625 3225 50  0001 C CNN
 F 3 "~" H 3625 3225 50  0001 C CNN
 F 4 "" H 3625 3225 50  0001 C CNN "Part"
@@
 $EndComp
 Text HLabel 4525 4075 2    50   Output ~ 0
-CT2
+CT3
 $Comp
 L Device:C_Small C?
@@
 F 0 "C25" H 3717 4471 50  0000 L CNN
 F 1 "100n" H 3717 4380 50  0000 L CNN
-F 2 "Capacitor_SMD:C_0805_2012Metric_Pad1.15x1.40mm_HandSolder" H 3625 4425 50  0001 C CNN
+F 2 "Capacitor_SMD:C_0805_2012Metric_Pad1.18x1.45mm_HandSolder" H 3625 4425 50  0001 C CNN
 F 3 "~" H 3625 4425 50  0001 C CNN
 F 4 "" H 3625 4425 50  0001 C CNN "Part"
@@
 	10725 3800 10525 3800
 Text Label 10525 3300 0    50   ~ 0
-CT0_L
+CT1_L
 Text Label 10525 3400 0    50   ~ 0
-CT0_K
+CT1_K
 Text Label 10525 3500 0    50   ~ 0
-CT1_L
+CT2_L
 Text Label 10525 3600 0    50   ~ 0
-CT1_K
+CT2_K
 Text Label 10525 3700 0    50   ~ 0
+CT3_L
+Text Label 10525 3800 0    50   ~ 0
+CT3_K
+Text Label 3075 2700 0    50   ~ 0
 CT2_L
-Text Label 10525 3800 0    50   ~ 0
+Text Label 2925 2700 2    50   ~ 0
 CT2_K
-Text Label 3075 1450 0    50   ~ 0
-CT0_L
-Text Label 2925 1450 2    50   ~ 0
-CT0_K
-Text Label 3075 2700 0    50   ~ 0
-CT1_L
-Text Label 2925 2700 2    50   ~ 0
-CT1_K
 Text Label 3075 3900 0    50   ~ 0
-CT2_L
+CT3_L
 Text Label 2925 3900 2    50   ~ 0
-CT2_K
+CT3_K
 $Comp
 L power:+3.3V #PWR042
@@
 CP_con
 Wire Wire Line
-	1825 6400 1825 6000
-Wire Wire Line
 	1825 6000 1975 6000
-Wire Wire Line
-	1825 6400 1475 6400
-Wire Wire Line
-	1825 6400 1825 6600
-Connection ~ 1825 6400
 Wire Wire Line
 	2475 6200 2225 6200
@@
 	2175 6000 2475 6000
 $Comp
-L Device:Opamp_Dual_Generic U11
+L agccs-ctrl22:Opamp_Dual_Generic_SmallVcc U11
 U 1 1 5E9126F4
 P 7900 1800
@@
 F 2 "atmevse-footprints:lv_screw_9pin_2" H 10925 3400 50  0001 C CNN
 F 3 "~" H 10925 3400 50  0001 C CNN
+F 4 " 490-TB004-508-18BE " H 10925 3400 50  0001 C CNN "PartNo"
 	1    10925 3400
 	1    0    0    -1
@@
 	1525 1925 2175 1925
 $Comp
-L agccs-ctrl22:12V_fused #PWR?
+L agccs-ctrl22:12V_fused #PWR0121
 U 1 1 6046C524
 P 10725 2550
-F 0 "#PWR?" H 10725 2400 50  0001 C CNN
+F 0 "#PWR0121" H 10725 2400 50  0001 C CNN
 F 1 "12V_fused" V 10740 2677 50  0000 L CNN
 F 2 "" H 10725 2550 50  0001 C CNN
@@
 	0    -1   -1   0
 $EndComp
+Wire Wire Line
+	1825 6000 1825 6600
+Text Label 2925 1450 2    50   ~ 0
+CT1_K
+Text Label 3075 1450 0    50   ~ 0
+CT1_L
+Text HLabel 1625 6000 0    50   Input ~ 0
+Signal_Relay
+Wire Wire Line
+	1825 6000 1625 6000
+Connection ~ 1825 6000
 $EndSCHEMATC
