File: circuit/KiCad/atmega4808_and_peripherals.sch (KiCad schematic (older format))
At the start: 34 parts, among them J3 Conn_01x04, J4 Conn_01x04, J5 Conn_02x04_Top_Bottom, Q1 BSS138, U10 ATmega4808-X, U7 SN65HVD72C, U8 FAN3214TMX, U9 ESP32-WROOM-32

Commit message: fx
Parts:
- removed D12: B220, Diode_SMD:D_SMB_Handsoldering, symbol Diode:B220
- added D12: PMEG4010BEA, Diode_SMD:D_SOD-323_HandSoldering, symbol Diode:PMEG4050EP
Changed lines of the file:
@@
 Wire Wire Line
 	1350 5750 1400 5750
-$Comp
-L Diode:B220 D12
-U 1 1 603DC56F
-P 850 5550
-F 0 "D12" H 850 5333 50  0000 C CNN
-F 1 "B220" H 850 5424 50  0000 C CNN
-F 2 "Diode_SMD:D_SMB_Handsoldering" H 850 5375 50  0001 C CNN
-F 3 "http://www.jameco.com/Jameco/Products/ProdDS/1538777.pdf" H 850 5550 50  0001 C CNN
-	1    850  5550
-	-1   0    0    1
-$EndComp
 Text Label 3250 5250 0    50   ~ 0
 12V_sep
@@
 Wire Wire Line
 	650  5550 650  5300
+$Comp
+L Diode:PMEG4050EP D?
+U 1 1 60368671
+P 850 5550
+AR Path="/5E98FA8A/60368671" Ref="D?"  Part="1"
+AR Path="/5E9B0066/60368671" Ref="D12"  Part="1"
+F 0 "D12" H 800 5400 50  0000 L CNN
+F 1 "PMEG4010BEA" H 450 5300 50  0000 L CNN
+F 2 "Diode_SMD:D_SOD-323_HandSoldering" H 850 5375 50  0001 C CNN
+F 3 "https://assets.nexperia.com/documents/data-sheet/PMEG4050EP.pdf" H 850 5550 50  0001 C CNN
+F 4 "" H 850 5550 50  0001 C CNN "Part"
+F 5 "771-PMEG4010BEA,135" H 850 5550 50  0001 C CNN "PartNo"
+F 6 "Mouser" H 850 5550 50  0001 C CNN "Supplier"
+	1    850  5550
+	-1   0    0    1
+$EndComp
 $EndSCHEMATC

Commit message: qe
Parts:
- removed C12: 10000u16V, Capacitor_THT:CP_Radial_D22.0mm_P10.00mm_SnapIn, symbol Device:CP_Small
- removed D12: PMEG4010BEA, Diode_SMD:D_SOD-323_HandSoldering, symbol Diode:PMEG4050EP
- removed R3, R4, R5, R6: 100, Resistor_SMD:R_0603_1608Metric_Pad1.05x0.95mm_HandSolder, symbol Device:R_Small
- added R41: 1k, symbol Device:R_Small
- R11: value 10k -> 2k
- R12: value 31.6k -> 5.6k
Connections:
- net labels added: +12P, BOT
- wire segments 183 -> 168
Other:
- moved on the sheet: C13, D2, D3, J3, U8

Commit message: qe
Parts:
- D2, D3, D4: PartNo 583-BAT54S -> 757-TBAT54SLM
- J4: PartNo (none) -> 710-61200821621; Supplier (none) -> Mouser
- R11: PartNo 594-MCT06030C1002FP5 -> 594-MCT06030C2001FP5
- R12: PartNo 594-MCT06030C3162FP5 -> 594-MCT06030C5601FP5
- R34, R37, R38: PartNo (none) -> 594-MCT06030C1001FP5; Supplier (none) -> Mouser
- R41: footprint (none) -> Resistor_SMD:R_0603_1608Metric_Pad1.05x0.95mm_HandSolder; PartNo (none) -> 594-MCT06030C1001FP5; Supplier (none) -> Mouser
- U10: PartNo (none) -> 556-ATMEGA4808-XF
Changed lines of the file:
@@
 F 0 "R41" V 6650 5000 50  0000 C CNN
 F 1 "1k" V 6650 4700 50  0000 C CNN
-F 2 "" H 6700 4850 50  0001 C CNN
+F 2 "Resistor_SMD:R_0603_1608Metric_Pad1.05x0.95mm_HandSolder" H 6700 4850 50  0001 C CNN
 F 3 "~" H 6700 4850 50  0001 C CNN
+F 4 "594-MCT06030C1001FP5" H 6700 4850 50  0001 C CNN "PartNo"
+F 5 "Mouser" H 6700 4850 50  0001 C CNN "Supplier"
 	1    6700 4850
 	0    1    1    0
@@
 F 2 "Resistor_SMD:R_0603_1608Metric_Pad1.05x0.95mm_HandSolder" H 9400 1300 50  0001 C CNN
 F 3 "~" H 9400 1300 50  0001 C CNN
+F 4 "594-MCT06030C1001FP5" H 9400 1300 50  0001 C CNN "PartNo"
+F 5 "Mouser" H 9400 1300 50  0001 C CNN "Supplier"
 	1    9400 1300
 	0    1    1    0
@@
 F 2 "Resistor_SMD:R_0603_1608Metric_Pad1.05x0.95mm_HandSolder" H 9400 1100 50  0001 C CNN
 F 3 "~" H 9400 1100 50  0001 C CNN
+F 4 "594-MCT06030C1001FP5" H 9400 1100 50  0001 C CNN "PartNo"
+F 5 "Mouser" H 9400 1100 50  0001 C CNN "Supplier"
 	1    9400 1100
 	0    1    1    0
@@
 F 2 "Resistor_SMD:R_0603_1608Metric_Pad1.05x0.95mm_HandSolder" H 9400 900 50  0001 C CNN
 F 3 "~" H 9400 900 50  0001 C CNN
+F 4 "594-MCT06030C1001FP5" H 9400 900 50  0001 C CNN "PartNo"
+F 5 "Mouser" H 9400 900 50  0001 C CNN "Supplier"
 	1    9400 900
 	0    1    1    0
@@
 F 2 "atmevse-footprints:UART0-Header" H 9300 1550 50  0001 C CNN
 F 3 "~" H 9300 1550 50  0001 C CNN
+F 4 "710-61200821621 " H 9300 1550 50  0001 C CNN "PartNo"
+F 5 "Mouser" H 9300 1550 50  0001 C CNN "Supplier"
 	1    9300 1550
 	1    0    0    -1
@@
 F 3 "~" H 8100 5200 50  0001 C CNN
 F 4 "" H 8100 5200 50  0001 C CNN "Part"
-F 5 "594-MCT06030C3162FP5" H 8100 5200 50  0001 C CNN "PartNo"
+F 5 "594-MCT06030C5601FP5 " H 8100 5200 50  0001 C CNN "PartNo"
 F 6 "Mouser" H 8100 5200 50  0001 C CNN "Supplier"
 	1    8100 5200
@@
 F 3 "~" H 7500 5950 50  0001 C CNN
 F 4 "" H 7500 5950 50  0001 C CNN "Part"
-F 5 "594-MCT06030C1002FP5 " H 7500 5950 50  0001 C CNN "PartNo"
+F 5 "594-MCT06030C2001FP5 " H 7500 5950 50  0001 C CNN "PartNo"
 F 6 "Mouser" H 7500 5950 50  0001 C CNN "Supplier"
 	1    7500 5950
@@
 F 3 "https://www.diodes.com/assets/Datasheets/ds11005.pdf" H 7680 5750 50  0001 C CNN
 F 4 "" H 7800 5750 50  0001 C CNN "Part"
-F 5 "583-BAT54S " H 7800 5750 50  0001 C CNN "PartNo"
+F 5 " 757-TBAT54SLM " H 7800 5750 50  0001 C CNN "PartNo"
 F 6 "Mouser" H 7800 5750 50  0001 C CNN "Supplier"
 	1    7800 5750
@@
 F 3 "https://www.diodes.com/assets/Datasheets/ds11005.pdf" H 4180 6450 50  0001 C CNN
 F 4 "" H 4300 6450 50  0001 C CNN "Part"
-F 5 "583-BAT54S " H 4300 6450 50  0001 C CNN "PartNo"
+F 5 " 757-TBAT54SLM " H 4300 6450 50  0001 C CNN "PartNo"
 F 6 "Mouser" H 4300 6450 50  0001 C CNN "Supplier"
 	1    4300 6450
@@
 F 3 "https://www.diodes.com/assets/Datasheets/ds11005.pdf" H 3680 6450 50  0001 C CNN
 F 4 "" H 3800 6450 50  0001 C CNN "Part"
-F 5 "583-BAT54S " H 3800 6450 50  0001 C CNN "PartNo"
+F 5 " 757-TBAT54SLM " H 3800 6450 50  0001 C CNN "PartNo"
 F 6 "Mouser" H 3800 6450 50  0001 C CNN "Supplier"
 	1    3800 6450
@@
 F 3 "http://ww1.microchip.com/downloads/en/DeviceDoc/40002018A.pdf" H 5750 3800 50  0001 C CNN
 F 4 "Mouser" H 5750 3800 50  0001 C CNN "Supplier"
+F 5 "556-ATMEGA4808-XF" H 5750 3800 50  0001 C CNN "PartNo"
 	1    5750 3800
 	1    0    0    -1

Commit message: qe
Parts:
- J4: PartNo 710-61200821621 -> (none)
- J5: value Conn_02x04_Top_Bottom -> Conn_02x04; symbol Connector_Generic:Conn_02x04_Top_Bottom -> Connector_Generic:Conn_02x04_Odd_Even; PartNo 710-61300821121 -> 710-61200821621
- U9: symbol RF_Module:ESP32-WROOM-32 -> RF_Module:ESP32-WROOM-32D
Changed lines of the file:
@@
 F 2 "atmevse-footprints:UART0-Header" H 9300 1550 50  0001 C CNN
 F 3 "~" H 9300 1550 50  0001 C CNN
-F 4 "710-61200821621 " H 9300 1550 50  0001 C CNN "PartNo"
+F 4 "" H 9300 1550 50  0001 C CNN "PartNo"
 F 5 "Mouser" H 9300 1550 50  0001 C CNN "Supplier"
 	1    9300 1550
@@
 $EndComp
 $Comp
-L Connector_Generic:Conn_02x04_Top_Bottom J5
+L Connector_Generic:Conn_02x04_Odd_Even J5
 U 1 1 5EC1F0B2
 P 9100 2100
 F 0 "J5" H 9150 1800 50  0000 C CNN
-F 1 "Conn_02x04_Top_Bottom" H 9150 2326 50  0000 C CNN
+F 1 "Conn_02x04" H 9150 2326 50  0000 C CNN
 F 2 "atmevse-footprints:PROGRAM-Header" H 9100 2100 50  0001 C CNN
 F 3 "~" H 9100 2100 50  0001 C CNN
 F 4 "" H 9100 2100 50  0001 C CNN "Part"
-F 5 "710-61300821121" H 9100 2100 50  0001 C CNN "PartNo"
+F 5 "710-61200821621 " H 9100 2100 50  0001 C CNN "PartNo"
 F 6 "Mouser" H 9100 2100 50  0001 C CNN "Supplier"
 	1    9100 2100
@@
 $EndComp
 $Comp
-L RF_Module:ESP32-WROOM-32 U9
+L RF_Module:ESP32-WROOM-32D U9
 U 1 1 5EC08E25
 P 9550 4400

Commit message: qe
Parts:
- U9: PartNo (none) -> 356-ESP32WRM32E128PH
Changed lines of the file:
@@
 F 3 "https://www.espressif.com/sites/default/files/documentation/esp32-wroom-32_datasheet_en.pdf" H 9250 4450 50  0001 C CNN
 F 4 "Mouser" H 9550 4400 50  0001 C CNN "Supplier"
+F 5 "356-ESP32WRM32E128PH " H 9550 4400 50  0001 C CNN "PartNo"
 	1    9550 4400
 	-1   0    0    -1

Commit message: qe
Parts:
- added D7: BAT54S, Package_TO_SOT_SMD:SOT-23_Handsoldering, symbol Diode:BAT54S
- added R24: 5.6k, Resistor_SMD:R_0603_1608Metric_Pad1.05x0.95mm_HandSolder, symbol Device:R_Small
- added R39: 2k, Resistor_SMD:R_0603_1608Metric_Pad1.05x0.95mm_HandSolder, symbol Device:R_Small
- C16: value 100u / 6.3V -> 100u6.3V
- C21: value 1n / 50V -> 1n50V
- C22: value 1u / 10V -> 1u10V
Connections:
- net labels added: 12V_buffered, AVR_RST, AVR_RX0, AVR_RX1, AVR_RX2, AVR_TX0, AVR_TX1, AVR_TX2, AVR_UDPI, ESP_EN, ESP_IO0
- net labels removed: +12P, 12V_sep, ATmega_RESET, ATmega_RX0, ATmega_RX2, ATmega_TX0, ATmega_TX2, ATmega_UDPI, EN, IO0, RS485_RX, RS485_TX
- wire segments 168 -> 187
Other:
- note added: "ATmega Extension Connector\n"
- note added: "ATmega/ESP Programming Header (Custom Pinout)\n"
- note added: "ATmega/ESP Serial Link\n(incl. Programming Atmega via J4)\n"
- note added: "Lock Driver\n"
- note added: "Operator Controls\n"
- note removed: "ATmega UART2 Connector\n"
- note removed: "ATmega UART:\n0 - PA0, PA1\n1 - PC0, PC1\n2 - PF0, PF1"
- note removed: "ATmega/ESP Programming & Serial Comms\n"
- note removed: "Lock Actuator Driver\n"
- moved on the sheet: C13, C14, C16, C21, C22, D2, D3, D4, J3, J4, J5, Q1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

Commit message: qe
Parts:
- C13, C14, C15, C17: footprint Capacitor_SMD:C_0805_2012Metric_Pad1.15x1.40mm_HandSolder -> Capacitor_SMD:C_0805_2012Metric_Pad1.18x1.45mm_HandSolder
Connections:
- net labels added: CT3
- net labels removed: CT0
Other:
- moved on the sheet: J4, R34
Changed lines of the file:
@@
 	5150 4700 5000 4700
 Text HLabel 5000 4400 0    50   Input ~ 0
-CT0
+CT1
 Text HLabel 5000 4550 0    50   Input ~ 0
-CT1
+CT2
 Text HLabel 5000 4700 0    50   Input ~ 0
-CT2
+CT3
 Text Label 5475 5950 2    50   ~ 0
 Lock_State
@@
 Text Label 5625 1325 0    50   ~ 0
 AVR_RST
-Wire Wire Line
-	6775 925  7375 925
 Wire Wire Line
 	6775 1125 7375 1125
@@
 U 1 1 5F47BE53
 P 6675 1325
-F 0 "R38" V 6625 1475 50  0000 C CNN
-F 1 "1k" V 6570 1325 50  0000 C CNN
+F 0 "R38" V 6600 1325 50  0000 C CNN
+F 1 "1k" V 6750 1325 50  0000 C CNN
 F 2 "Resistor_SMD:R_0603_1608Metric_Pad1.05x0.95mm_HandSolder" H 6675 1325 50  0001 C CNN
 F 3 "~" H 6675 1325 50  0001 C CNN
@@
 U 1 1 5F47BC59
 P 6675 1125
-F 0 "R37" V 6625 1275 50  0000 C CNN
-F 1 "1k" V 6570 1125 50  0000 C CNN
+F 0 "R37" V 6625 975 50  0000 C CNN
+F 1 "1k" V 6625 1250 50  0000 C CNN
 F 2 "Resistor_SMD:R_0603_1608Metric_Pad1.05x0.95mm_HandSolder" H 6675 1125 50  0001 C CNN
 F 3 "~" H 6675 1125 50  0001 C CNN
@@
 L Device:R_Small R34
 U 1 1 5F47B25C
-P 6675 925
-F 0 "R34" V 6625 1075 50  0000 C CNN
-F 1 "1k" V 6570 925 50  0000 C CNN
-F 2 "Resistor_SMD:R_0603_1608Metric_Pad1.05x0.95mm_HandSolder" H 6675 925 50  0001 C CNN
-F 3 "~" H 6675 925 50  0001 C CNN
-F 4 "594-MCT06030C1001FP5" H 6675 925 50  0001 C CNN "PartNo"
-F 5 "Mouser" H 6675 925 50  0001 C CNN "Supplier"
-	1    6675 925
+P 6125 925
+F 0 "R34" V 6050 925 50  0000 C CNN
+F 1 "1k" V 6200 925 50  0000 C CNN
+F 2 "Resistor_SMD:R_0603_1608Metric_Pad1.05x0.95mm_HandSolder" H 6125 925 50  0001 C CNN
+F 3 "~" H 6125 925 50  0001 C CNN
+F 4 "594-MCT06030C1001FP5" H 6125 925 50  0001 C CNN "PartNo"
+F 5 "Mouser" H 6125 925 50  0001 C CNN "Supplier"
+	1    6125 925
 	0    1    1    0
 $EndComp
@@
 F 0 "C13" H 1092 5771 50  0000 L CNN
 F 1 "100n" V 1100 5525 50  0000 L CNN
-F 2 "Capacitor_SMD:C_0805_2012Metric_Pad1.15x1.40mm_HandSolder" H 1000 5725 50  0001 C CNN
+F 2 "Capacitor_SMD:C_0805_2012Metric_Pad1.18x1.45mm_HandSolder" H 1000 5725 50  0001 C CNN
 F 3 "~" H 1000 5725 50  0001 C CNN
 F 4 "" H 1000 5725 50  0001 C CNN "Part"
@@
 F 0 "C14" V 2954 1425 50  0000 C CNN
 F 1 "100n" V 2863 1425 50  0000 C CNN
-F 2 "Capacitor_SMD:C_0805_2012Metric_Pad1.15x1.40mm_HandSolder" H 2725 1425 50  0001 C CNN
+F 2 "Capacitor_SMD:C_0805_2012Metric_Pad1.18x1.45mm_HandSolder" H 2725 1425 50  0001 C CNN
 F 3 "~" H 2725 1425 50  0001 C CNN
 F 4 "" H 2725 1425 50  0001 C CNN "Part"
@@
 F 0 "C15" V 5521 5000 50  0000 C CNN
 F 1 "100n" V 5612 5000 50  0000 C CNN
-F 2 "Capacitor_SMD:C_0805_2012Metric_Pad1.15x1.40mm_HandSolder" H 5750 5000 50  0001 C CNN
+F 2 "Capacitor_SMD:C_0805_2012Metric_Pad1.18x1.45mm_HandSolder" H 5750 5000 50  0001 C CNN
 F 3 "~" H 5750 5000 50  0001 C CNN
 F 4 "" H 5750 5000 50  0001 C CNN "Part"
@@
 F 0 "C17" H 7392 4046 50  0000 L CNN
 F 1 "100n" H 7392 3955 50  0000 L CNN
-F 2 "Capacitor_SMD:C_0805_2012Metric_Pad1.15x1.40mm_HandSolder" H 7300 4000 50  0001 C CNN
+F 2 "Capacitor_SMD:C_0805_2012Metric_Pad1.18x1.45mm_HandSolder" H 7300 4000 50  0001 C CNN
 F 3 "~" H 7300 4000 50  0001 C CNN
 F 4 "" H 7300 4000 50  0001 C CNN "Part"
@@
 L Connector_Generic:Conn_01x04 J4
 U 1 1 5F466074
-P 6675 1700
-F 0 "J4" H 6675 1925 50  0000 C CNN
-F 1 "Conn_01x04" H 6975 1600 50  0001 C CNN
-F 2 "atmevse-footprints:UART0-Header" H 6675 1700 50  0001 C CNN
-F 3 "~" H 6675 1700 50  0001 C CNN
-F 4 "" H 6675 1700 50  0001 C CNN "PartNo"
-F 5 "Mouser" H 6675 1700 50  0001 C CNN "Supplier"
-	1    6675 1700
+P 7100 1700
+F 0 "J4" H 7100 1925 50  0000 C CNN
+F 1 "Conn_01x04" H 7400 1600 50  0001 C CNN
+F 2 "atmevse-footprints:UART0-Header" H 7100 1700 50  0001 C CNN
+F 3 "~" H 7100 1700 50  0001 C CNN
+F 4 "" H 7100 1700 50  0001 C CNN "PartNo"
+F 5 "Mouser" H 7100 1700 50  0001 C CNN "Supplier"
+	1    7100 1700
 	1    0    0    1
 $EndComp
@@
 $EndComp
 Wire Wire Line
-	5625 1125 6275 1125
-Wire Wire Line
-	5625 1325 6375 1325
-Wire Wire Line
-	6475 1800 6300 1800
-Wire Wire Line
-	6475 1500 6375 1500
-Wire Wire Line
-	6375 1500 6375 1325
-Connection ~ 6375 1325
-Wire Wire Line
-	6375 1325 6575 1325
-Wire Wire Line
-	6275 1600 6275 1125
-Connection ~ 6275 1125
-Wire Wire Line
-	6275 1125 6575 1125
-Wire Wire Line
-	6475 1700 6175 1700
-Wire Wire Line
-	6175 1700 6175 925
-Wire Wire Line
-	5625 925  6175 925
-Connection ~ 6175 925
-Wire Wire Line
-	6175 925  6575 925
-Wire Wire Line
-	6275 1600 6475 1600
+	6900 1800 6300 1800
+Wire Wire Line
+	6900 1500 6500 1500
+Wire Wire Line
+	6900 1700 6300 1700
+Wire Wire Line
+	6400 1600 6900 1600
 Wire Notes Line
 	4225 525  5425 525
@@
 Operator Controls\n
 $Comp
-L agccs-ctrl22:12V_buffered #PWR?
+L agccs-ctrl22:12V_buffered #PWR0120
 U 1 1 60462D21
 P 1000 5300
-F 0 "#PWR?" H 1000 5150 50  0001 C CNN
+F 0 "#PWR0120" H 1000 5150 50  0001 C CNN
 F 1 "12V_buffered" H 1075 5450 50  0000 C CNN
 F 2 "" H 1000 5300 50  0001 C CNN
@@
 	1    0    0    -1
 $EndComp
+Wire Wire Line
+	5625 925  6025 925
+Wire Wire Line
+	5625 1125 6400 1125
+Wire Wire Line
+	5625 1325 6500 1325
+Wire Wire Line
+	6500 1500 6500 1325
+Connection ~ 6500 1325
+Wire Wire Line
+	6500 1325 6575 1325
+Wire Wire Line
+	6300 1700 6300 925
+Wire Wire Line
+	6225 925  6300 925
+Connection ~ 6300 925
+Wire Wire Line
+	6300 925  7375 925
+Wire Wire Line
+	6400 1600 6400 1125
+Connection ~ 6400 1125
+Wire Wire Line
+	6400 1125 6575 1125
 $EndSCHEMATC
