File: circuit/KiCad/mains_and_power.sch (KiCad schematic (older format))
At the start: 29 parts, among them J1 Screw_Terminal_01x05, J2 Screw_Terminal_01x05, U1 AQH3223, U2 AQH3223, U3 AQH3223, U4 IRM-10-12, U5 TC7660SEOA, U6 AP5100

Commit message: qe
Parts:
- added C12: 10000u16V, Capacitor_THT:CP_Radial_D22.0mm_P10.00mm_SnapIn, symbol Device:CP_Small
- added C27: 2200u16V, Capacitor_THT:CP_Radial_D12.5mm_P7.50mm, symbol Device:CP_Small
- added D12: PMEG4010BEA, Diode_SMD:D_SOD-323_HandSoldering, symbol Diode:PMEG4050EP
- added D13: 9.1, Diode_SMD:D_SOD-323_HandSoldering, symbol Device:D_Zener_Small_ALT
- added R3, R4, R5, R6: 100, Resistor_SMD:R_0603_1608Metric_Pad1.05x0.95mm_HandSolder, symbol Device:R_Small
- added R40: 2k, Resistor_SMD:R_0603_1608Metric_Pad1.05x0.95mm_HandSolder, symbol Device:R_Small
Connections:
- net +12V: now also C27.1, D12.2 (A), D13.1 (K)
- net GND: now also C12.2, C27.2, R40.2
- new net: D12.1 (K), R3.2, R4.2, R5.2, R6.2
- new net +12P: C12.1, R3.1, R4.1, R5.1, R6.1
- new net BOT: D13.2 (A), R40.1
Other:
- moved on the sheet: C1, C10, C11, C2, C26, C3, C4, C5, C6, C7, C8, C9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

Commit message: qe
Parts:
- C12: value 10000u16V -> 15000u16V; PartNo 871-B41231A4109M000 -> 871-B41231A4159M000
- R40: PartNo (none) -> 594-MCT06030C2001FP5; Supplier (none) -> Mouser
Changed lines of the file:
@@
 F 2 "Resistor_SMD:R_0603_1608Metric_Pad1.05x0.95mm_HandSolder" V 5480 5600 50  0001 C CNN
 F 3 "~" H 5550 5600 50  0001 C CNN
+F 4 "594-MCT06030C2001FP5 " H 5550 5600 50  0001 C CNN "PartNo"
+F 5 "Mouser" H 5550 5600 50  0001 C CNN "Supplier"
 	1    5550 5600
 	1    0    0    -1
@@
 AR Path="/5E98FA8A/60BEF32A" Ref="C12"  Part="1"
 F 0 "C12" H 7288 5246 50  0000 L CNN
-F 1 "10000u16V" V 7050 4950 50  0000 L CNN
+F 1 "15000u16V" V 7050 4950 50  0000 L CNN
 F 2 "Capacitor_THT:CP_Radial_D22.0mm_P10.00mm_SnapIn" H 7200 5200 50  0001 C CNN
 F 3 "~" H 7200 5200 50  0001 C CNN
 F 4 "" H 7200 5200 50  0001 C CNN "Part"
-F 5 "871-B41231A4109M000" H 7200 5200 50  0001 C CNN "PartNo"
+F 5 "871-B41231A4159M000" H 7200 5200 50  0001 C CNN "PartNo"
 F 6 "Mouser" H 7200 5200 50  0001 C CNN "Supplier"
 	1    7200 5200

Commit message: qe
Parts:
- added F1: FSMD020, Fuse:Fuse_1812_4532Metric_Pad1.30x3.40mm_HandSolder, symbol Device:Polyfuse_Small
- renumbered RV3 to RV1, RV1 to RV3
Connections:
- net +12V: now also F1.1
- net L_fused: now reaches F2.1, U1.6 (DS3), U2.6 (DS3), U3.6 (DS3), U4.2 (AC/L)
- net +12P renamed 12V_buffered
- new net 12V_fused: F1.2
Other:
- moved on the sheet: C1, C10, C11, C12, C2, C26, C27, C3, C4, C5, C6, C7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

Commit message: qe
Parts:
- C1, C10, C11, C2, C3, C4, C5, C6, C7, C8, C9: footprint Capacitor_SMD:C_0805_2012Metric_Pad1.15x1.40mm_HandSolder -> Capacitor_SMD:C_0805_2012Metric_Pad1.18x1.45mm_HandSolder
- J2: PartNo (none) -> 490-TB005-762-10BE
Changed lines of the file:
@@
 F 0 "C1" H 6575 1750 50  0000 L CNN
 F 1 "10u16V" V 6625 1400 50  0000 L CNN
-F 2 "Capacitor_SMD:C_0805_2012Metric_Pad1.15x1.40mm_HandSolder" H 6563 1500 50  0001 C CNN
+F 2 "Capacitor_SMD:C_0805_2012Metric_Pad1.18x1.45mm_HandSolder" H 6563 1500 50  0001 C CNN
 F 3 "~" H 6525 1650 50  0001 C CNN
 F 4 "" H 6525 1650 50  0001 C CNN "Part"
@@
 F 0 "C3" H 6925 1750 50  0000 L CNN
 F 1 "10u16V" V 6975 1400 50  0000 L CNN
-F 2 "Capacitor_SMD:C_0805_2012Metric_Pad1.15x1.40mm_HandSolder" H 6913 1500 50  0001 C CNN
+F 2 "Capacitor_SMD:C_0805_2012Metric_Pad1.18x1.45mm_HandSolder" H 6913 1500 50  0001 C CNN
 F 3 "~" H 6875 1650 50  0001 C CNN
 F 4 "" H 6875 1650 50  0001 C CNN "Part"
@@
 F 0 "C6" H 7625 1750 50  0000 L CNN
 F 1 "10u16V" V 7675 1400 50  0000 L CNN
-F 2 "Capacitor_SMD:C_0805_2012Metric_Pad1.15x1.40mm_HandSolder" H 7613 1500 50  0001 C CNN
+F 2 "Capacitor_SMD:C_0805_2012Metric_Pad1.18x1.45mm_HandSolder" H 7613 1500 50  0001 C CNN
 F 3 "~" H 7575 1650 50  0001 C CNN
 F 4 "" H 7575 1650 50  0001 C CNN "Part"
@@
 F 0 "C7" H 7800 1750 50  0000 L CNN
 F 1 "100n" V 7825 1475 50  0000 L CNN
-F 2 "Capacitor_SMD:C_0805_2012Metric_Pad1.15x1.40mm_HandSolder" H 7963 1500 50  0001 C CNN
+F 2 "Capacitor_SMD:C_0805_2012Metric_Pad1.18x1.45mm_HandSolder" H 7963 1500 50  0001 C CNN
 F 3 "~" H 7925 1650 50  0001 C CNN
 F 4 "" H 7925 1650 50  0001 C CNN "Part"
@@
 F 0 "C9" V 9096 1350 50  0000 C CNN
 F 1 "100n" V 9187 1350 50  0000 C CNN
-F 2 "Capacitor_SMD:C_0805_2012Metric_Pad1.15x1.40mm_HandSolder" H 9325 1350 50  0001 C CNN
+F 2 "Capacitor_SMD:C_0805_2012Metric_Pad1.18x1.45mm_HandSolder" H 9325 1350 50  0001 C CNN
 F 3 "~" H 9325 1350 50  0001 C CNN
 F 4 "" H 9325 1350 50  0001 C CNN "Part"
@@
 F 0 "C10" H 10375 1750 50  0000 L CNN
 F 1 "10u16V" V 10425 1350 50  0000 L CNN
-F 2 "Capacitor_SMD:C_0805_2012Metric_Pad1.15x1.40mm_HandSolder" H 10563 1500 50  0001 C CNN
+F 2 "Capacitor_SMD:C_0805_2012Metric_Pad1.18x1.45mm_HandSolder" H 10563 1500 50  0001 C CNN
 F 3 "~" H 10525 1650 50  0001 C CNN
 F 4 "" H 10525 1650 50  0001 C CNN "Part"
@@
 F 0 "C11" H 10675 1750 50  0000 L CNN
 F 1 "10u16V" V 10725 1350 50  0000 L CNN
-F 2 "Capacitor_SMD:C_0805_2012Metric_Pad1.15x1.40mm_HandSolder" H 10863 1500 50  0001 C CNN
+F 2 "Capacitor_SMD:C_0805_2012Metric_Pad1.18x1.45mm_HandSolder" H 10863 1500 50  0001 C CNN
 F 3 "~" H 10825 1650 50  0001 C CNN
 F 4 "" H 10825 1650 50  0001 C CNN "Part"
@@
 F 0 "C4" H 8880 3376 50  0000 L CNN
 F 1 "100n" V 8915 3130 50  0000 L CNN
-F 2 "Capacitor_SMD:C_0805_2012Metric_Pad1.15x1.40mm_HandSolder" H 8803 3180 50  0001 C CNN
+F 2 "Capacitor_SMD:C_0805_2012Metric_Pad1.18x1.45mm_HandSolder" H 8803 3180 50  0001 C CNN
 F 3 "~" H 8765 3330 50  0001 C CNN
 F 4 "" H 8765 3330 50  0001 C CNN "Part"
@@
 F 0 "C2" H 8305 3865 50  0000 L CNN
 F 1 "10u16V" V 8525 3595 50  0000 L CNN
-F 2 "Capacitor_SMD:C_0805_2012Metric_Pad1.15x1.40mm_HandSolder" H 8453 3630 50  0001 C CNN
+F 2 "Capacitor_SMD:C_0805_2012Metric_Pad1.18x1.45mm_HandSolder" H 8453 3630 50  0001 C CNN
 F 3 "~" H 8415 3780 50  0001 C CNN
 F 4 "" H 8415 3780 50  0001 C CNN "Part"
@@
 F 0 "C8" H 10730 4176 50  0000 L CNN
 F 1 "10u16V" V 10765 3830 50  0000 L CNN
-F 2 "Capacitor_SMD:C_0805_2012Metric_Pad1.15x1.40mm_HandSolder" H 10653 3980 50  0001 C CNN
+F 2 "Capacitor_SMD:C_0805_2012Metric_Pad1.18x1.45mm_HandSolder" H 10653 3980 50  0001 C CNN
 F 3 "~" H 10615 4130 50  0001 C CNN
 F 4 "" H 10615 4130 50  0001 C CNN "Part"
@@
 F 0 "C5" H 7325 1750 50  0000 L CNN
 F 1 "10u16V" V 7375 1400 50  0000 L CNN
-F 2 "Capacitor_SMD:C_0805_2012Metric_Pad1.15x1.40mm_HandSolder" H 7263 1500 50  0001 C CNN
+F 2 "Capacitor_SMD:C_0805_2012Metric_Pad1.18x1.45mm_HandSolder" H 7263 1500 50  0001 C CNN
 F 3 "~" H 7225 1650 50  0001 C CNN
 F 4 "" H 7225 1650 50  0001 C CNN "Part"
@@
 L power:PWR_FLAG #FLG?
 U 1 1 60BB0926
-P 2000 7175
+P 3000 7175
 AR Path="/60BB0926" Ref="#FLG?"  Part="1"
 AR Path="/5E98FA8A/60BB0926" Ref="#FLG0101"  Part="1"
-F 0 "#FLG0101" H 2000 7250 50  0001 C CNN
-F 1 "PWR_FLAG" H 2000 7348 50  0000 C CNN
-F 2 "" H 2000 7175 50  0001 C CNN
-F 3 "~" H 2000 7175 50  0001 C CNN
-	1    2000 7175
+F 0 "#FLG0101" H 3000 7250 50  0001 C CNN
+F 1 "PWR_FLAG" H 3000 7348 50  0000 C CNN
+F 2 "" H 3000 7175 50  0001 C CNN
+F 3 "~" H 3000 7175 50  0001 C CNN
+	1    3000 7175
 	-1   0    0    1
 $EndComp
@@
 L power:-12V #PWR0110
 U 1 1 60BC5A0D
-P 2500 7025
-F 0 "#PWR0110" H 2500 7125 50  0001 C CNN
-F 1 "-12V" H 2515 7198 50  0000 C CNN
-F 2 "" H 2500 7025 50  0001 C CNN
-F 3 "" H 2500 7025 50  0001 C CNN
-	1    2500 7025
+P 3500 7025
+F 0 "#PWR0110" H 3500 7125 50  0001 C CNN
+F 1 "-12V" H 3515 7198 50  0000 C CNN
+F 2 "" H 3500 7025 50  0001 C CNN
+F 3 "" H 3500 7025 50  0001 C CNN
+	1    3500 7025
 	1    0    0    -1
 $EndComp
@@
 L power:+3.3V #PWR0111
 U 1 1 60BCCB52
-P 2000 7025
-F 0 "#PWR0111" H 2000 6875 50  0001 C CNN
-F 1 "+3.3V" H 2015 7198 50  0000 C CNN
-F 2 "" H 2000 7025 50  0001 C CNN
-F 3 "" H 2000 7025 50  0001 C CNN
-	1    2000 7025
-	1    0    0    -1
-$EndComp
-Wire Wire Line
-	2000 7025 2000 7175
+P 3000 7025
+F 0 "#PWR0111" H 3000 6875 50  0001 C CNN
+F 1 "+3.3V" H 3015 7198 50  0000 C CNN
+F 2 "" H 3000 7025 50  0001 C CNN
+F 3 "" H 3000 7025 50  0001 C CNN
+	1    3000 7025
+	1    0    0    -1
+$EndComp
+Wire Wire Line
+	3000 7025 3000 7175
 Wire Notes Line
 	11125 550  11125 2400
@@
 	7300 5625 7300 6000
 Wire Wire Line
-	2500 7025 2500 7175
+	3500 7025 3500 7175
 $Comp
 L power:PWR_FLAG #FLG?
 U 1 1 60BB780A
-P 2500 7175
+P 3500 7175
 AR Path="/60BB780A" Ref="#FLG?"  Part="1"
 AR Path="/5E98FA8A/60BB780A" Ref="#FLG0102"  Part="1"
-F 0 "#FLG0102" H 2500 7250 50  0001 C CNN
-F 1 "PWR_FLAG" H 2500 7348 50  0000 C CNN
-F 2 "" H 2500 7175 50  0001 C CNN
-F 3 "~" H 2500 7175 50  0001 C CNN
-	1    2500 7175
+F 0 "#FLG0102" H 3500 7250 50  0001 C CNN
+F 1 "PWR_FLAG" H 3500 7348 50  0000 C CNN
+F 2 "" H 3500 7175 50  0001 C CNN
+F 3 "~" H 3500 7175 50  0001 C CNN
+	1    3500 7175
 	-1   0    0    1
 $EndComp
@@
 F 2 "atmevse-footprints:hv_screw_5pin_2" H 775 2150 50  0001 C CNN
 F 3 "~" H 775 2150 50  0001 C CNN
+F 4 " 490-TB005-762-10BE " H 775 2150 50  0001 C CNN "PartNo"
 	1    775  2150
 	-1   0    0    -1
@@
 	5450 4975 5450 5025
 $Comp
-L agccs-ctrl22:12V_buffered #PWR?
+L agccs-ctrl22:12V_buffered #PWR0113
 U 1 1 60477EB6
 P 7300 4700
-F 0 "#PWR?" H 7300 4550 50  0001 C CNN
+F 0 "#PWR0113" H 7300 4550 50  0001 C CNN
 F 1 "12V_buffered" H 7315 4873 50  0000 C CNN
 F 2 "" H 7300 4700 50  0001 C CNN
@@
 	1    0    0    -1
 $EndComp
+$Comp
+L power:PWR_FLAG #FLG?
+U 1 1 6048F56E
+P 2000 7175
+AR Path="/6048F56E" Ref="#FLG?"  Part="1"
+AR Path="/5E98FA8A/6048F56E" Ref="#FLG0104"  Part="1"
+F 0 "#FLG0104" H 2000 7250 50  0001 C CNN
+F 1 "PWR_FLAG" H 2000 7348 50  0000 C CNN
+F 2 "" H 2000 7175 50  0001 C CNN
+F 3 "~" H 2000 7175 50  0001 C CNN
+	1    2000 7175
+	-1   0    0    1
+$EndComp
+Wire Wire Line
+	2000 7025 2000 7175
+$Comp
+L power:PWR_FLAG #FLG?
+U 1 1 604991E2
+P 2500 7175
+AR Path="/604991E2" Ref="#FLG?"  Part="1"
+AR Path="/5E98FA8A/604991E2" Ref="#FLG0106"  Part="1"
+F 0 "#FLG0106" H 2500 7250 50  0001 C CNN
+F 1 "PWR_FLAG" H 2500 7348 50  0000 C CNN
+F 2 "" H 2500 7175 50  0001 C CNN
+F 3 "~" H 2500 7175 50  0001 C CNN
+	1    2500 7175
+	-1   0    0    1
+$EndComp
+Wire Wire Line
+	2500 7025 2500 7175
+$Comp
+L agccs-ctrl22:12V_buffered #PWR0122
+U 1 1 604CBE12
+P 2500 7025
+F 0 "#PWR0122" H 2500 6875 50  0001 C CNN
+F 1 "12V_buffered" H 2515 7198 50  0000 C CNN
+F 2 "" H 2500 7025 50  0001 C CNN
+F 3 "" H 2500 7025 50  0001 C CNN
+	1    2500 7025
+	1    0    0    -1
+$EndComp
+$Comp
+L agccs-ctrl22:12V_fused #PWR0123
+U 1 1 604CCDE8
+P 2000 7025
+F 0 "#PWR0123" H 2000 6875 50  0001 C CNN
+F 1 "12V_fused" H 2015 7198 50  0000 C CNN
+F 2 "" H 2000 7025 50  0001 C CNN
+F 3 "" H 2000 7025 50  0001 C CNN
+	1    2000 7025
+	1    0    0    -1
+$EndComp
