File: circuit/Rev-1-2/analog_section_low_voltage.sch (KiCad schematic (older format))
At the start: 37 parts, among them J6 Screw_Terminal_01x09, J7 Screw_Terminal_01x09, U11 LM7332, U12 CPC1114N, U13 CPC1114N, U14 LM321LV

Commit message: qe
Parts:
- D10, D5, D8, D9: PartNo 757-TBAT54SLM -> 757-TBAT54SLM
- J6: PartNo na -> (none)
- J7: PartNo 490-TB004-508-18BE -> 490-TB004-508-18BE
Changed lines of the file:
@@
 F 3 "https://www.diodes.com/assets/Datasheets/ds11005.pdf" H 8030 4725 50  0001 C CNN
 F 4 "" H 8150 4725 50  0001 C CNN "Part"
-F 5 "757-TBAT54SLM " H 8150 4725 50  0001 C CNN "PartNo"
+F 5 " 757-TBAT54SLM " H 8150 4725 50  0001 C CNN "PartNo"
 F 6 "Mouser" H 8150 4725 50  0001 C CNN "Supplier"
 	1    8150 4725
@@
 F 2 "atmevse-footprints:lv_screw_9pin_1" H 10925 2450 50  0001 C CNN
 F 3 "~" H 10925 2450 50  0001 C CNN
-F 4 "na" H 10925 2450 50  0001 C CNN "PartNo"
 	1    10925 2450
 	1    0    0    -1
@@
 F 2 "atmevse-footprints:lv_screw_9pin_2" H 10925 3400 50  0001 C CNN
 F 3 "~" H 10925 3400 50  0001 C CNN
-F 4 "490-TB004-508-18BE " H 10925 3400 50  0001 C CNN "PartNo"
+F 4 " 490-TB004-508-18BE " H 10925 3400 50  0001 C CNN "PartNo"
 	1    10925 3400
 	1    0    0    -1
@@
 F 2 "Package_TO_SOT_SMD:SOT-23_Handsoldering" H 4275 2100 50  0001 L CNN
 F 3 "https://www.diodes.com/assets/Datasheets/ds11005.pdf" H 4080 1975 50  0001 C CNN
-F 4 "757-TBAT54SLM " H 4200 1975 50  0001 C CNN "PartNo"
+F 4 " 757-TBAT54SLM " H 4200 1975 50  0001 C CNN "PartNo"
 F 5 "Mouser" H 4200 1975 50  0001 C CNN "Supplier"
 	1    4200 1975
@@
 F 2 "Package_TO_SOT_SMD:SOT-23_Handsoldering" H 4275 3350 50  0001 L CNN
 F 3 "https://www.diodes.com/assets/Datasheets/ds11005.pdf" H 4080 3225 50  0001 C CNN
-F 4 "757-TBAT54SLM " H 4200 3225 50  0001 C CNN "PartNo"
+F 4 " 757-TBAT54SLM " H 4200 3225 50  0001 C CNN "PartNo"
 F 5 "Mouser" H 4200 3225 50  0001 C CNN "Supplier"
 	1    4200 3225
@@
 F 2 "Package_TO_SOT_SMD:SOT-23_Handsoldering" H 4275 4550 50  0001 L CNN
 F 3 "https://www.diodes.com/assets/Datasheets/ds11005.pdf" H 4080 4425 50  0001 C CNN
-F 4 "757-TBAT54SLM " H 4200 4425 50  0001 C CNN "PartNo"
+F 4 " 757-TBAT54SLM " H 4200 4425 50  0001 C CNN "PartNo"
 F 5 "Mouser" H 4200 4425 50  0001 C CNN "Supplier"
 	1    4200 4425
