File: circuit/Rev-1-2/atmega4808_and_peripherals.sch (KiCad schematic (older format))
At the start: 32 parts, among them J3 Conn_01x04, J4 Conn_01x04, J5 Conn_02x04, Q1 BSS138, U10 ATmega4808-X, U7 SN65HVD72C, U8 FAN3214TMX, U9 ESP32-WROOM-32

Commit message: qe
Parts:
- D2, D3, D4, D7: PartNo 757-TBAT54SLM -> 757-TBAT54SLM
- J4: PartNo na -> (none)
Changed lines of the file:
@@
 F 3 "https://www.diodes.com/assets/Datasheets/ds11005.pdf" H 3330 6400 50  0001 C CNN
 F 4 "" H 3450 6400 50  0001 C CNN "Part"
-F 5 "757-TBAT54SLM " H 3450 6400 50  0001 C CNN "PartNo"
+F 5 " 757-TBAT54SLM " H 3450 6400 50  0001 C CNN "PartNo"
 F 6 "Mouser" H 3450 6400 50  0001 C CNN "Supplier"
 	1    3450 6400
@@
 F 3 "https://www.diodes.com/assets/Datasheets/ds11005.pdf" H 2830 6400 50  0001 C CNN
 F 4 "" H 2950 6400 50  0001 C CNN "Part"
-F 5 "757-TBAT54SLM " H 2950 6400 50  0001 C CNN "PartNo"
+F 5 " 757-TBAT54SLM " H 2950 6400 50  0001 C CNN "PartNo"
 F 6 "Mouser" H 2950 6400 50  0001 C CNN "Supplier"
 	1    2950 6400
@@
 F 2 "atmevse-footprints:UART0-Header" H 7100 1700 50  0001 C CNN
 F 3 "~" H 7100 1700 50  0001 C CNN
-F 4 "na" H 7100 1700 50  0001 C CNN "PartNo"
+F 4 "" H 7100 1700 50  0001 C CNN "PartNo"
 F 5 "Mouser" H 7100 1700 50  0001 C CNN "Supplier"
 	1    7100 1700
@@
 F 3 "https://www.diodes.com/assets/Datasheets/ds11005.pdf" H 5055 6500 50  0001 C CNN
 F 4 "" H 5175 6500 50  0001 C CNN "Part"
-F 5 "757-TBAT54SLM " H 5175 6500 50  0001 C CNN "PartNo"
+F 5 " 757-TBAT54SLM " H 5175 6500 50  0001 C CNN "PartNo"
 F 6 "Mouser" H 5175 6500 50  0001 C CNN "Supplier"
 	1    5175 6500
@@
 F 3 "https://www.diodes.com/assets/Datasheets/ds11005.pdf" H 1905 4100 50  0001 C CNN
 F 4 "" H 2025 4100 50  0001 C CNN "Part"
-F 5 "757-TBAT54SLM " H 2025 4100 50  0001 C CNN "PartNo"
+F 5 " 757-TBAT54SLM " H 2025 4100 50  0001 C CNN "PartNo"
 F 6 "Mouser" H 2025 4100 50  0001 C CNN "Supplier"
 	1    2025 4100
