File: circuit/Rev-1-2/mains_and_power.sch (KiCad schematic (older format))
At the start: 39 parts, among them J1 Screw_Terminal_01x05, J2 Screw_Terminal_01x05, U1 AQH3223, U2 AQH3223, U3 AQH3223, U4 IRM-10-12, U5 TC7660SEOA, U6 AP5100

Commit message: qe
Parts:
- J1: PartNo na -> (none)
Changed lines of the file:
@@
 F 2 "atmevse-footprints:hv_screw_5pin_1" H 775 1600 50  0001 C CNN
 F 3 "~" H 775 1600 50  0001 C CNN
-F 4 "na" H 775 1600 50  0001 C CNN "PartNo"
 	1    775  1600
 	-1   0    0    -1
