File: circuit/j5adaptor/agccs-j5adaptor-1-2.sch (KiCad schematic (older format))
At the start: 12 parts, among them J5 Conn_02x04_Odd_Even

Commit message: qe
Parts:
- added R?: 120, symbol Device:R
Connections:
- net at J5.6 (Pin_6): now also R?.1; no longer JP?.2
- new net: JP?.2, R?.2
Other:
- note added: "*** ESP serial line programming: hold down ESP_BOOT while cycling ESP_EN;\nstart “make flash” before releasing ESP_BOOT; on the AGCCS board, \nESP_BOOT is BLACK and ESP_EN is GREY"
- note added: "*** when pulled to ground, our firmeware “demesh.c”\nwill boot into target-debug mode (i.e. accespoint with telnet\nforwarding of the AVRs Tx0 und Rx0); cycle EPS_EN to\ntrigger re-boot."
- note removed: "*** ESP serial line programming: hold down ESP_BOOT while cycling ESP_EN;\non the AGCCS board, ESP_BOOT is BLACK and ESP_EN is GREY"
- note removed: "*** when pulled to ground, our firmeware “demesh.c”\nwill go in target-debug mode (i.e. accespoint with telnet\nforwarding of the AVRs Tx0 und Rx0)"
Changed lines of the file:
@@
 	6850 1750 7400 1750
-Wire Wire Line
-	7400 1750 7400 3525
 Wire Wire Line
 	7400 3725 7400 4150
@@
 Text Notes 3450 2650 0    59   ~ 0
 *** keep unattained to pass on serial line to ESP \n(programming and monitoring)\n*** hold down for UPDI programming the AVR with \nPyupdi (the ESP will then lalso listen to the UPDI \nprogramming protocol, but this does not matter)\n*** on the AGCCS board, this is the RED switch
-Text Notes 4675 3775 0    59   ~ 0
-*** when pulled to ground, our firmeware “demesh.c”\nwill go in target-debug mode (i.e. accespoint with telnet\nforwarding of the AVRs Tx0 und Rx0)
-Text Notes 6350 4425 0    59   ~ 0
-*** ESP serial line programming: hold down ESP_BOOT while cycling ESP_EN;\non the AGCCS board, ESP_BOOT is BLACK and ESP_EN is GREY
+Text Notes 4525 3775 0    59   ~ 0
+*** when pulled to ground, our firmeware “demesh.c”\nwill boot into target-debug mode (i.e. accespoint with telnet\nforwarding of the AVRs Tx0 und Rx0); cycle  EPS_EN to\ntrigger re-boot.
+Text Notes 6375 4500 0    59   ~ 0
+*** ESP serial line programming: hold down ESP_BOOT while cycling ESP_EN;\nstart “make flash” before releasing ESP_BOOT; on the AGCCS board, \nESP_BOOT is BLACK and ESP_EN is GREY
+$Comp
+L Device:R R?
+U 1 1 604BA489
+P 7400 3175
+F 0 "R?" H 7470 3221 50  0001 L CNN
+F 1 "120" H 7330 3175 50  0000 R CNN
+F 2 "" V 7330 3175 50  0001 C CNN
+F 3 "~" H 7400 3175 50  0001 C CNN
+	1    7400 3175
+	-1   0    0    -1
+$EndComp
+Wire Wire Line
+	7400 3325 7400 3525
+Wire Wire Line
+	7400 3025 7400 1750
 $EndSCHEMATC

Commit message: qe
Connections:
- net at J?.3 (RxD), R?.1: now also SW?.2 (B)
Other:
- note added: "*** we use a USB-to-Serial converter \nwith a CP102 chip from Silicon Labs; it \nis fast and reliable. \n*** double check the output voltage … \nmust not be more than 3.3V (!)"
Changed lines of the file:
@@
 	5200 1650 6350 1650
-Wire Wire Line
-	4175 1750 3700 1750
 Wire Wire Line
 	5350 1750 5350 1450
@@
 	6850 1850 8375 1850
 Wire Wire Line
-	2475 4150 7400 4150
+	3000 4150 7400 4150
 Wire Wire Line
-	2475 1850 2350 1850
-Wire Wire Line
-	2475 1850 2475 4150
+	3000 1850 2350 1850
 Wire Wire Line
 	9150 3325 9150 3425
@@
 Wire Wire Line
 	7400 3025 7400 1750
+Wire Wire Line
+	3700 1750 4200 1750
+Wire Wire Line
+	3000 1850 3000 4150
+Text Notes 900  2625 0    59   ~ 0
+*** we  use a USB-to-Serial converter \nwith a  CP102 chip from Silicon Labs; it \nis fast and reliable. \n*** double check the output voltage … \nmust not be more than 3.3V (!)
 $EndSCHEMATC

Commit message: qe
Connections:
- net ESP_IO15: now reaches J5.6 (Pin_6), R?.1
Other:
- note added: "*** ESP serial line programming: hold down ESP_BOOT while cycling ESP_EN;\nstart “make flash” before releasing ESP_BOOT; on the AGCCS board, \nESP_EN is BLACK and ESP_BOOT is GREY"
- note added: "*** when pulled to ground, our firmeware “demesh.c”\nwill boot into target-debug mode (i.e. accespoint with telnet\nforwarding of the AVRs Tx0 und Rx0); cycle EPS_EN to\ntrigger re-boot. (OPTIONAL — you may prefer to use a plain\njumper wire from ESP_IO15 to GND directly)"
- note added: "OPTIONAL LED: show blink \ncodes from demesh.c"
- note removed: "*** ESP serial line programming: hold down ESP_BOOT while cycling ESP_EN;\nstart “make flash” before releasing ESP_BOOT; on the AGCCS board, \nESP_BOOT is BLACK and ESP_EN is GREY"
- note removed: "*** when pulled to ground, our firmeware “demesh.c”\nwill boot into target-debug mode (i.e. accespoint with telnet\nforwarding of the AVRs Tx0 und Rx0); cycle EPS_EN to\ntrigger re-boot."
Changed lines of the file:
@@
 *** keep unattained to pass on serial line to ESP \n(programming and monitoring)\n*** hold down for UPDI programming the AVR with \nPyupdi (the ESP will then lalso listen to the UPDI \nprogramming protocol, but this does not matter)\n*** on the AGCCS board, this is the RED switch
 Text Notes 4525 3775 0    59   ~ 0
-*** when pulled to ground, our firmeware “demesh.c”\nwill boot into target-debug mode (i.e. accespoint with telnet\nforwarding of the AVRs Tx0 und Rx0); cycle  EPS_EN to\ntrigger re-boot.
+*** when pulled to ground, our firmeware “demesh.c”\nwill boot into target-debug mode (i.e. accespoint with telnet\nforwarding of the AVRs Tx0 und Rx0); cycle  EPS_EN to\ntrigger re-boot. (OPTIONAL — you may prefer to use a plain\njumper wire from ESP_IO15 to GND directly)
 Text Notes 6375 4500 0    59   ~ 0
-*** ESP serial line programming: hold down ESP_BOOT while cycling ESP_EN;\nstart “make flash” before releasing ESP_BOOT; on the AGCCS board, \nESP_BOOT is BLACK and ESP_EN is GREY
+*** ESP serial line programming: hold down ESP_BOOT while cycling ESP_EN;\nstart “make flash” before releasing ESP_BOOT; on the AGCCS board, \nESP_EN is BLACK and ESP_BOOT is GREY
 $Comp
 L Device:R R?
@@
 Text Notes 900  2625 0    59   ~ 0
 *** we  use a USB-to-Serial converter \nwith a  CP102 chip from Silicon Labs; it \nis fast and reliable. \n*** double check the output voltage … \nmust not be more than 3.3V (!)
+Text Label 6875 1750 0    59   ~ 0
+ESP_IO15
+Wire Notes Line
+	8900 1700 9475 1700
+Wire Notes Line
+	9475 1700 9475 2650
+Wire Notes Line
+	8900 1700 8900 2650
+Wire Notes Line
+	8900 2650 9475 2650
+Text Notes 8775 1450 0    59   ~ 0
+OPTIONAL LED: show blink \ncodes from demesh.c
 $EndSCHEMATC
